Commit message: 2024-4-26 10:15 新的URDF模型重新训练

File: resources/robots/ZQ_Humanoid/urdf/ZQ_Humanoid.urdf (robot description, URDF)
Before this commit: robot ZQ_Humanoid, 13 links, 12 joints
Links:
- link Y4: mass 2.9408 -> 2.72497
- link Z4: mass 3.15 -> 2.72510

File: resources/robots/ZQ_Humanoid/urdf/ZQ_Humanoid_long_foot.urdf (robot description, URDF)
Before this commit: robot ZQ_Humanoid, 13 links, 12 joints
Links:
- link Y4: mass 2.9408 -> 2.72497
- link Z4: mass 3.15 -> 2.72510
