Commit message: 2024-5-7 18:14 步态生成改成星动纪元原版.

File: resources/robots/ZQ_Humanoid/urdf/ZQ_Humanoid_long_foot.urdf (robot description, URDF)
Before this commit: robot ZQ_Humanoid, 13 links, 12 joints
Links:
- link Y3: geometry collision box size=0.1 0.1 0.25; visual mesh filename=../meshes/RightLeg_Link_03.STL
- link Y4: geometry collision box size=0.05 0.05 0.30; visual mesh filename=../meshes/RightLeg_Link_04.STL
- link Z3: geometry collision box size=0.1 0.1 0.25; visual mesh filename=../meshes/LeftLeg_Link_03.STL
- link Z4: geometry collision box size=0.05 0.05 0.30; visual mesh filename=../meshes/LeftLeg_Link_04.STL

Commit message: 2024-5-9 11:15 按唐博建议改了resample时count不重置为0。加了一些初始随机化的开关。play时加了1秒站立姿态。

File: resources/robots/ZQ_Humanoid/urdf/ZQ_Humanoid_long_foot.urdf (robot description, URDF)
Before this commit: robot ZQ_Humanoid, 13 links, 12 joints
Links:
- link Y3: geometry collision box size=0.08 0.08 0.25; visual mesh filename=../meshes/RightLeg_Link_03.STL
- link Z3: geometry collision box size=0.08 0.08 0.25; visual mesh filename=../meshes/LeftLeg_Link_03.STL
