Commit message: 2024-5-10 9：47 5dof线足模型训练

File: resources/robots/ZQ_Humanoid/urdf/ZQ_Humanoid_10dof.urdf (robot description, URDF)
Before this commit: robot zq01, 11 links, 10 joints
Links:
- link Y3: geometry collision box size=0.08 0.08 0.25; visual mesh filename=../meshes/RightLeg_Link_03.STL
- link Y4: geometry collision box size=0.05 0.05 0.30; visual mesh filename=../meshes/RightLeg_Link_04.STL
- link Z3: geometry collision box size=0.08 0.08 0.25; visual mesh filename=../meshes/LeftLeg_Link_03.STL
- link Z4: geometry collision box size=0.05 0.05 0.30; visual mesh filename=../meshes/LeftLeg_Link_04.STL

Commit message: 2024-5-10 12:00 修复了线足5DOF和板足6DOF不同的地方

File: resources/robots/ZQ_Humanoid/urdf/ZQ_Humanoid_10dof.urdf (robot description, URDF)
Before this commit: robot zq01, 11 links, 10 joints
Links:
- link Y5: geometry collision cylinder length=0.24 radius=0.02; visual mesh filename=../meshes/RightLeg_Link_SingleDOF_05.STL
- link Z5: geometry collision cylinder length=0.24 radius=0.02; visual mesh filename=../meshes/LeftLeg_Link_SingleDOF_05.STL
